File: hardware/tiliqua-motherboard/encoder.kicad_sch (KiCad schematic)
At the start: 10 parts, among them SW3 RotaryEncoder_Switch

Commit message: * start adding DVI redriver
Changed lines of the file:
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@@
 (kicad_sch
-	(version 20231120)
+	(version 20250114)
 	(generator "eeschema")
-	(generator_version "8.0")
+	(generator_version "9.0")
 	(paper "A4")
 	(junction
@@
 		(shape output)
 		(at 170.18 83.82 0)
-		(fields_autoplaced yes)
 		(effects
 			(font
@@
 		(shape output)
 		(at 170.18 86.36 0)
-		(fields_autoplaced yes)
 		(effects
 			(font
@@
 		(shape output)
 		(at 170.18 67.31 0)
-		(fields_autoplaced yes)
 		(effects
 			(font
